File: hardware/mainboard/focusbot_mainboard.kicad_pcb (KiCad board)
At the start: 2 copper layers, 64 x 70 mm, 52 parts, among them Q1 AO3401A, SW1 Power_Switch, U1 ESP32-S3-WROOM-1-N16R8, U2 TP4056, U3 DW01A, U4 FS8205A, U5 SY8089AAAC, U6 DRV8833PWP, U7 MAX98357A, U8 MPU-6050

Commit message: feat(branding): rename project to FocusBot, clean up CAD/KiCad artifacts, add photorealistic 3D renders to README
Other:
- board text added: "FOCUSBOT MAINBOARD v12.0"
- board text added: "OPEN-SOURCE HARDWARE • CERN-OHL-S"
Changed lines of the file:
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@@
 	)
 	(embedded_fonts no)
+	(gr_text "FOCUSBOT MAINBOARD v12.0"
+		(at 150 128)
+		(layer "F.SilkS")
+		(uuid "fbc-mb-title-01")
+		(effects
+			(font
+				(size 1.2 1.2)
+				(thickness 0.2)
+			)
+			(justify center)
+		)
+	)
+	(gr_text "OPEN-SOURCE HARDWARE • CERN-OHL-S"
+		(at 150 131)
+		(layer "F.SilkS")
+		(uuid "fbc-mb-oshw-01")
+		(effects
+			(font
+				(size 0.9 0.9)
+				(thickness 0.15)
+			)
+			(justify center)
+		)
+	)
 )

Commit message: fix(pcb): repair KiCad 10 syntax errors & feat(firmware): complete FocusBot v12.0 ESP32-S3 firmware
Other:
- board text added: "OPEN-SOURCE HARDWARE - CERN-OHL-S"
- board text removed: "OPEN-SOURCE HARDWARE • CERN-OHL-S"
Changed lines of the file:
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@@
 		(layer "Edge.Cuts")
 	)
+	(gr_text "OPEN-SOURCE HARDWARE - CERN-OHL-S"
+		(at 150 131 0)
+		(layer "F.SilkS")
+		(effects
+			(font
+				(size 0.9 0.9)
+				(thickness 0.15)
+			)
+		)
+	)
+	(gr_text "FOCUSBOT MAINBOARD v12.0"
+		(at 150 128 0)
+		(layer "F.SilkS")
+		(effects
+			(font
+				(size 1.2 1.2)
+				(thickness 0.2)
+			)
+		)
+	)
 	(segment
 		(start 128.225 114)
@@
 	)
 	(embedded_fonts no)
-	(gr_text "FOCUSBOT MAINBOARD v12.0"
-		(at 150 128)
-		(layer "F.SilkS")
-		(uuid "fbc-mb-title-01")
-		(effects
-			(font
-				(size 1.2 1.2)
-				(thickness 0.2)
-			)
-			(justify center)
-		)
-	)
-	(gr_text "OPEN-SOURCE HARDWARE • CERN-OHL-S"
-		(at 150 131)
-		(layer "F.SilkS")
-		(uuid "fbc-mb-oshw-01")
-		(effects
-			(font
-				(size 0.9 0.9)
-				(thickness 0.15)
-			)
-			(justify center)
-		)
-	)
 )

Commit message: fix(pcb): clear keepout zone 100% and reroute 3V3 trace under RF shield
Routing:
- net 3V3: track 173.4 -> 170.0 mm, vias 0 -> 2
Other:
- board text removed: "OPEN-SOURCE HARDWARE - CERN-OHL-S"
Changed lines of the file:
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@@
 			(polygon
 				(pts
-					(xy 126 77.25) (xy 174 77.25) (xy 174 56.25) (xy 126 56.25)
+					(xy 140 77) (xy 160 77) (xy 160 65) (xy 140 65)
 				)
 			)
@@
 		)
 		(fp_text user "${REFERENCE}"
-			(at 0 0 0)
+			(at 0 -9.5 0)
 			(unlocked yes)
 			(layer "F.Fab")
@@
 		(layer "Edge.Cuts")
 	)
-	(gr_text "OPEN-SOURCE HARDWARE - CERN-OHL-S"
-		(at 150 131 0)
-		(layer "F.SilkS")
-		(effects
-			(font
-				(size 0.9 0.9)
-				(thickness 0.15)
-			)
-		)
-	)
 	(gr_text "FOCUSBOT MAINBOARD v12.0"
-		(at 150 128 0)
+		(at 153 132.5 0)
 		(layer "F.SilkS")
 		(effects
@@
 	)
 	(segment
+		(start 167.82 77)
+		(end 165.5 78.5)
+		(width 0.45)
+		(layer "F.Cu")
+		(net "3V3")
+	)
+	(segment
 		(start 143.7204 105.867)
 		(end 143.3563 105.5029)
@@
 	)
 	(segment
+		(start 143.5 78.5)
+		(end 141.25 80.01)
+		(width 0.45)
+		(layer "F.Cu")
+		(net "3V3")
+	)
+	(segment
 		(start 172.1126 97.4638)
 		(end 167.6941 93.0453)
@@
 	)
 	(segment
-		(start 167.825 74.6296)
-		(end 164.0587 70.8633)
-		(width 0.45)
-		(layer "F.Cu")
-		(net "3V3")
-	)
-	(segment
-		(start 167.825 77)
-		(end 167.825 74.6296)
-		(width 0.45)
-		(layer "F.Cu")
-		(net "3V3")
-	)
-	(segment
 		(start 145.7833 105.1264)
 		(end 145.0427 105.867)
@@
 	)
 	(segment
-		(start 164.0587 70.8633)
-		(end 153.7889 70.8633)
-		(width 0.45)
-		(layer "F.Cu")
-		(net "3V3")
-	)
-	(segment
-		(start 153.7889 70.8633)
-		(end 144.6422 80.01)
-		(width 0.45)
-		(layer "F.Cu")
-		(net "3V3")
-	)
-	(segment
 		(start 167.225 128.5)
 		(end 165.3524 130.3726)
@@
 		(net "3V3")
 	)
+	(via
+		(at 143.5 78.5)
+		(size 0.6)
+		(drill 0.3)
+		(layers "F.Cu" "B.Cu")
+		(net "3V3")
+	)
+	(via
+		(at 165.5 78.5)
+		(size 0.6)
+		(drill 0.3)
+		(layers "F.Cu" "B.Cu")
+		(net "3V3")
+	)
+	(segment
+		(start 165.5 78.5)
+		(end 143.5 78.5)
+		(width 0.45)
+		(layer "B.Cu")
+		(net "3V3")
+	)
